File: zero-hm-10-breakout/zero-hm-10-breakout.brd (EAGLE design)
At the start: 25.1 x 34.3 mm, 9 parts, among them U1 HM-10

Commit message: first working routing
Parts:
- removed D1: BLUE, SparkFun-LED:LED-0603
- added PWR: BLU, adafruit:CHIPLED_0805
- RXD: value GREEN -> GRN; device SparkFun-LED:LED-0603 -> adafruit:CHIPLED_0805
- TXD: device SparkFun-LED:LED-0603 -> adafruit:CHIPLED_0805
- moved R3 31.8 mm to (17.8, 31.8), turned to 180 degrees
- moved R1 22.2 mm to (21.6, 11.4)
- moved RXD 21.6 mm to (21.6, 15.2), turned to 180 degrees
- moved TXD 14.5 mm to (21.6, 22.9), turned to 180 degrees
- moved R2 14.2 mm to (21.6, 19.1)
- moved R4 10.2 mm to (7.62, 31.8), turned to 0 degrees
Connections:
- net GND: now also PWR.C; no longer D1.C
- net N$3: now also PWR.A; no longer D1.A
Routing:
- net GND: track 0.00 -> 50.6 mm
- net VDD: track 0.00 -> 29.9 mm, vias 0 -> 1
- net RX: track 0.00 -> 27.4 mm, vias 0 -> 1
- net TX: track 0.00 -> 24.7 mm, vias 0 -> 1
- net N$3: track 0.00 -> 3.13 mm

Commit message: good layout
Parts:
- moved R4 28.4 mm to (2.54, 3.81), turned to 90 degrees
- moved RXD 17.3 mm to (16.5, 31.8), turned to 0 degrees
- moved R2 16.3 mm to (11.4, 31.8)
- moved R3 13.0 mm to (5.08, 29.2), turned to 90 degrees
- moved TXD 11.7 mm to (14.0, 31.8)
- moved R1 7.73 mm to (22.9, 3.81)
- moved PWR 3.81 mm to (8.89, 31.8), turned to 180 degrees
Routing:
- net GND: track 50.6 -> 93.0 mm, vias 0 -> 2
- net N$2: track 0.00 -> 30.1 mm
- net N$5: track 0.00 -> 29.6 mm
- net TX: track 24.7 -> 47.8 mm, vias 1 -> 2
- net VDD: track 29.9 -> 52.2 mm
- net RX: track 27.4 -> 43.9 mm
- net N$4: track 0.00 -> 6.99 mm
- net N$1: track 0.00 -> 3.13 mm
- net N$3: track 3.13 -> 6.20 mm

Commit message: better board layout
Parts:
- turned RXD to 180 degrees
Routing:
- net GND: track 93.0 -> 54.3 mm, vias 2 -> 1
- net RX: track 43.9 -> 50.4 mm
- net TX: track 47.8 -> 41.4 mm
- net N$2: track 30.1 -> 31.2 mm, vias 0 -> 2
- net VDD: track 52.2 -> 52.7 mm, vias 1 -> 2
Changed lines of the file:
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@@
 <attribute name="PROD_ID" value="RES-11622" x="40.64" y="46.99" size="1.778" layer="27" rot="R90" display="off"/>
 </element>
-<element name="RXD" library="adafruit" package="CHIPLED_0805" value="GRN" x="16.51" y="31.75"/>
-<element name="TXD" library="adafruit" package="CHIPLED_0805" value="RED" x="13.97" y="31.75" rot="R180"/>
-<element name="PWR" library="adafruit" package="CHIPLED_0805" value="BLU" x="8.89" y="31.75" rot="R180"/>
+<element name="RXD" library="adafruit" package="CHIPLED_0805" value="GRN" x="16.51" y="31.75" smashed="yes" rot="R180">
+<attribute name="NAME" x="17.78" y="33.02" size="0.3048" layer="25" rot="R270"/>
+<attribute name="VALUE" x="17.78" y="31.75" size="0.3048" layer="27" rot="R270"/>
+</element>
+<element name="TXD" library="adafruit" package="CHIPLED_0805" value="RED" x="13.97" y="31.75" smashed="yes" rot="R180">
+<attribute name="NAME" x="15.24" y="33.02" size="0.3048" layer="25" rot="R270"/>
+<attribute name="VALUE" x="15.24" y="31.75" size="0.3048" layer="27" rot="R270"/>
+</element>
+<element name="PWR" library="adafruit" package="CHIPLED_0805" value="BLU" x="8.89" y="31.75" smashed="yes" rot="R180">
+<attribute name="NAME" x="7.62" y="33.02" size="0.3048" layer="25" rot="R270"/>
+<attribute name="VALUE" x="10.16" y="33.02" size="0.3048" layer="27" rot="R270"/>
+</element>
 </elements>
 <signals>
@@
 <contactref element="TXD" pad="C"/>
 <contactref element="PWR" pad="C"/>
-<wire x1="19.05" y1="27.94" x2="17.78" y2="29.21" width="0.254" layer="1"/>
-<wire x1="19.05" y1="26.67" x2="19.05" y2="27.94" width="0.254" layer="1"/>
+<wire x1="16.51" y1="30.48" x2="13.97" y2="30.48" width="0.254" layer="1"/>
+<wire x1="13.97" y1="30.48" x2="13.97" y2="30.7" width="0.254" layer="1"/>
+<wire x1="16.51" y1="30.48" x2="17.78" y2="29.21" width="0.254" layer="1"/>
+<wire x1="16.51" y1="30.48" x2="16.51" y2="30.7" width="0.254" layer="1"/>
+<wire x1="17.78" y1="27.94" x2="19.05" y2="26.67" width="0.254" layer="1"/>
+<wire x1="17.78" y1="29.21" x2="17.78" y2="27.94" width="0.254" layer="1"/>
 <wire x1="17.78" y1="29.21" x2="17.93" y2="28.96" width="0.254" layer="1"/>
 <wire x1="7.62" y1="29.21" x2="8.89" y2="30.48" width="0.254" layer="1"/>
@@
 <wire x1="7.62" y1="29.21" x2="7.62" y2="27.94" width="0.254" layer="1"/>
 <wire x1="7.62" y1="29.21" x2="7.43" y2="28.96" width="0.254" layer="1"/>
+<wire x1="8.89" y1="8.89" x2="1.27" y2="8.89" width="0.254" layer="16"/>
+<wire x1="8.89" y1="24.13" x2="8.89" y2="8.89" width="0.254" layer="1"/>
+<wire x1="6.35" y1="26.67" x2="8.89" y2="24.13" width="0.254" layer="1"/>
+<wire x1="1.27" y1="8.89" x2="1.7" y2="8.35" width="0.254" layer="16"/>
 <wire x1="6.35" y1="26.67" x2="19.05" y2="26.67" width="0.254" layer="1"/>
 <wire x1="19.05" y1="26.67" x2="19.47" y2="26.89" width="0.254" layer="1"/>
-<wire x1="16.51" y1="33.02" x2="15.24" y2="31.75" width="0.254" layer="1"/>
-<wire x1="15.24" y1="31.75" x2="13.97" y2="30.48" width="0.254" layer="1"/>
-<wire x1="13.97" y1="30.48" x2="13.97" y2="30.7" width="0.254" layer="1"/>
-<wire x1="16.51" y1="33.02" x2="16.51" y2="32.8" width="0.254" layer="1"/>
-<wire x1="20.32" y1="26.67" x2="15.24" y2="31.75" width="0.254" layer="16"/>
-<wire x1="20.32" y1="7.62" x2="20.32" y2="26.67" width="0.254" layer="16"/>
-<wire x1="2.54" y1="7.62" x2="8.89" y2="7.62" width="0.254" layer="16"/>
-<wire x1="8.89" y1="7.62" x2="20.32" y2="7.62" width="0.254" layer="16"/>
-<wire x1="1.27" y1="8.89" x2="2.54" y2="7.62" width="0.254" layer="16"/>
-<wire x1="1.27" y1="8.89" x2="1.7" y2="8.35" width="0.254" layer="16"/>
-<wire x1="8.89" y1="24.13" x2="6.35" y2="26.67" width="0.254" layer="1"/>
-<wire x1="8.89" y1="7.62" x2="8.89" y2="24.13" width="0.254" layer="1"/>
 <wire x1="6.35" y1="26.67" x2="5.93" y2="26.89" width="0.254" layer="1"/>
-<via x="15.24" y="31.75" extent="1-16" drill="0.6096"/>
-<via x="8.89" y="7.62" extent="1-16" drill="0.6096"/>
+<via x="8.89" y="8.89" extent="1-16" drill="0.6096"/>
 </signal>
 <signal name="VDD">
@@
 <contactref element="R4" pad="2"/>
 <wire x1="15.24" y1="5.08" x2="2.54" y2="5.08" width="0.254" layer="1"/>
-<wire x1="15.24" y1="22.86" x2="15.24" y2="5.08" width="0.254" layer="1"/>
-<wire x1="17.78" y1="25.4" x2="15.24" y2="22.86" width="0.254" layer="1"/>
-<wire x1="19.05" y1="25.4" x2="17.78" y2="25.4" width="0.254" layer="1"/>
+<wire x1="15.24" y1="21.59" x2="15.24" y2="5.08" width="0.254" layer="1"/>
+<wire x1="19.05" y1="25.4" x2="15.24" y2="21.59" width="0.254" layer="1"/>
 <wire x1="2.54" y1="5.08" x2="2.54" y2="4.71" width="0.254" layer="1"/>
 <wire x1="19.05" y1="25.4" x2="19.47" y2="25.39" width="0.254" layer="1"/>
-<wire x1="2.54" y1="25.4" x2="1.27" y2="26.67" width="0.254" layer="16"/>
-<wire x1="12.7" y1="25.4" x2="2.54" y2="25.4" width="0.254" layer="16"/>
-<wire x1="15.24" y1="22.86" x2="12.7" y2="25.4" width="0.254" layer="1"/>
-<wire x1="1.27" y1="26.67" x2="1.7" y2="26.35" width="0.254" layer="16"/>
-<via x="12.7" y="25.4" extent="1-16" drill="0.6096"/>
+<wire x1="3.81" y1="24.13" x2="1.27" y2="26.67" width="0.254" layer="1"/>
+<wire x1="3.81" y1="22.86" x2="3.81" y2="24.13" width="0.254" layer="1"/>
+<wire x1="5.08" y1="21.59" x2="3.81" y2="22.86" width="0.254" layer="16"/>
+<wire x1="15.24" y1="21.59" x2="5.08" y2="21.59" width="0.254" layer="16"/>
+<wire x1="1.27" y1="26.67" x2="1.7" y2="26.35" width="0.254" layer="1"/>
+<via x="3.81" y="22.86" extent="1-16" drill="0.6096"/>
+<via x="15.24" y="21.59" extent="1-16" drill="0.6096"/>
 </signal>
 <signal name="TX">
@@
 <contactref element="U$1" pad="3"/>
 <contactref element="R2" pad="1"/>
-<wire x1="12.7" y1="31.75" x2="11.43" y2="30.48" width="0.254" layer="1"/>
-<wire x1="19.05" y1="25.4" x2="12.7" y2="31.75" width="0.254" layer="16"/>
-<wire x1="19.05" y1="22.86" x2="19.05" y2="25.4" width="0.254" layer="16"/>
-<wire x1="1.27" y1="22.86" x2="17.78" y2="22.86" width="0.254" layer="16"/>
-<wire x1="17.78" y1="22.86" x2="19.05" y2="22.86" width="0.254" layer="16"/>
+<wire x1="10.16" y1="31.75" x2="11.43" y2="30.48" width="0.254" layer="1"/>
+<wire x1="10.16" y1="24.13" x2="10.16" y2="31.75" width="0.254" layer="16"/>
+<wire x1="3.81" y1="24.13" x2="10.16" y2="24.13" width="0.254" layer="16"/>
+<wire x1="2.54" y1="22.86" x2="3.81" y2="24.13" width="0.254" layer="16"/>
+<wire x1="1.27" y1="22.86" x2="2.54" y2="22.86" width="0.254" layer="16"/>
 <wire x1="11.43" y1="30.48" x2="11.43" y2="30.85" width="0.254" layer="1"/>
 <wire x1="1.27" y1="22.86" x2="1.7" y2="22.35" width="0.254" layer="16"/>
-<wire x1="17.78" y1="8.89" x2="19.47" y2="8.89" width="0.254" layer="1"/>
-<wire x1="17.78" y1="22.86" x2="17.78" y2="8.89" width="0.254" layer="16"/>
-<via x="12.7" y="31.75" extent="1-16" drill="0.6096"/>
-<via x="17.78" y="8.89" extent="1-16" drill="0.6096"/>
+<wire x1="16.51" y1="11.43" x2="19.05" y2="8.89" width="0.254" layer="1"/>
+<wire x1="16.51" y1="21.59" x2="16.51" y2="11.43" width="0.254" layer="1"/>
+<wire x1="13.97" y1="24.13" x2="16.51" y2="21.59" width="0.254" layer="16"/>
+<wire x1="10.16" y1="24.13" x2="13.97" y2="24.13" width="0.254" layer="16"/>
+<wire x1="19.05" y1="8.89" x2="19.47" y2="8.89" width="0.254" layer="1"/>
+<via x="10.16" y="31.75" extent="1-16" drill="0.6096"/>
+<via x="16.51" y="21.59" extent="1-16" drill="0.6096"/>
 </signal>
 <signal name="RX">
@@
 <contactref element="U$1" pad="2"/>
 <contactref element="R1" pad="1"/>
-<wire x1="16.51" y1="8.89" x2="22.86" y2="2.54" width="0.254" layer="1"/>
-<wire x1="17.78" y1="10.16" x2="16.51" y2="8.89" width="0.254" layer="1"/>
-<wire x1="19.05" y1="10.16" x2="17.78" y2="10.16" width="0.254" layer="1"/>
+<wire x1="21.59" y1="3.81" x2="22.86" y2="2.54" width="0.254" layer="1"/>
+<wire x1="21.59" y1="8.89" x2="21.59" y2="3.81" width="0.254" layer="1"/>
+<wire x1="20.32" y1="10.16" x2="21.59" y2="8.89" width="0.254" layer="1"/>
+<wire x1="19.05" y1="10.16" x2="20.32" y2="10.16" width="0.254" layer="1"/>
 <wire x1="22.86" y1="2.54" x2="22.86" y2="2.91" width="0.254" layer="1"/>
+<wire x1="10.16" y1="33.02" x2="1.27" y2="24.13" width="0.254" layer="16"/>
+<wire x1="17.78" y1="25.4" x2="10.16" y2="33.02" width="0.254" layer="16"/>
+<wire x1="17.78" y1="11.43" x2="17.78" y2="25.4" width="0.254" layer="16"/>
+<wire x1="19.05" y1="10.16" x2="17.78" y2="11.43" width="0.254" layer="1"/>
+<wire x1="1.27" y1="24.13" x2="1.7" y2="24.35" width="0.254" layer="16"/>
 <wire x1="19.05" y1="10.16" x2="19.47" y2="10.39" width="0.254" layer="1"/>
-<wire x1="17.78" y1="24.13" x2="1.27" y2="24.13" width="0.254" layer="16"/>
-<wire x1="17.78" y1="10.16" x2="17.78" y2="24.13" width="0.254" layer="1"/>
-<wire x1="1.27" y1="24.13" x2="1.7" y2="24.35" width="0.254" layer="16"/>
-<via x="17.78" y="24.13" extent="1-16" drill="0.6096"/>
+<via x="17.78" y="11.43" extent="1-16" drill="0.6096"/>
 </signal>
 <signal name="N$1">
@@
 <contactref element="R1" pad="2"/>
 <contactref element="RXD" pad="A"/>
-<wire x1="21.59" y1="6.35" x2="22.86" y2="5.08" width="0.254" layer="1"/>
-<wire x1="21.59" y1="27.94" x2="21.59" y2="6.35" width="0.254" layer="1"/>
-<wire x1="19.05" y1="30.48" x2="21.59" y2="27.94" width="0.254" layer="1"/>
-<wire x1="16.51" y1="30.48" x2="19.05" y2="30.48" width="0.254" layer="1"/>
-<wire x1="22.86" y1="5.08" x2="22.86" y2="4.71" width="0.254" layer="1"/>
-<wire x1="16.51" y1="30.48" x2="16.51" y2="30.7" width="0.254" layer="1"/>
+<wire x1="22.86" y1="6.35" x2="22.86" y2="4.71" width="0.254" layer="1"/>
+<wire x1="19.05" y1="10.16" x2="22.86" y2="6.35" width="0.254" layer="16"/>
+<wire x1="19.05" y1="30.48" x2="19.05" y2="10.16" width="0.254" layer="16"/>
+<wire x1="16.51" y1="33.02" x2="19.05" y2="30.48" width="0.254" layer="1"/>
+<wire x1="16.51" y1="33.02" x2="16.51" y2="32.8" width="0.254" layer="1"/>
+<via x="22.86" y="6.35" extent="1-16" drill="0.6096"/>
+<via x="19.05" y="30.48" extent="1-16" drill="0.6096"/>
 </signal>
 <signal name="N$3">
