File: zero-hm-10-breakout/zero-hm-10-breakout.sch (EAGLE design)
At the start: 2 parts, among them U1 HM-10

Commit message: just about todo routing
Parts:
- added D1: BLUE, SparkFun-LED:LED-BLUE0603
- added R1, R2, R3, R4: 470R, SparkFun-Resistors:0.3OHM-1/8W-1%(0805)
- added RXD: GREEN, SparkFun-LED:LED-GREEN0603
- added TXD: RED, SparkFun-LED:LED-GREEN0603
Connections:
- new net N$1: R2.2, TXD.A
- new net N$2: R1.2, RXD.A
- new net N$3: D1.A, R3.2
- new net N$4: R3.1, U1.P1_2
- new net N$5: R4.1, U1.P1_3
- new net RX: R1.1, U$1.DOUT, U1.P1_7
- new net TX: R2.1, U$1.DIN, U1.P1_6
- net GND: now also D1.C, RXD.C, TXD.C, U1.GND@4
- net VDD: now also R4.2
Changed lines of the file:
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@@
 <setting verticaltext="up"/>
 </settings>
-<grid distance="0.05" unitdist="inch" unit="inch" style="lines" multiple="1" display="yes" altdistance="0.025" altunitdist="inch" altunit="inch"/>
+<grid distance="0.05" unitdist="inch" unit="inch" style="lines" multiple="1" display="no" altdistance="0.025" altunitdist="inch" altunit="inch"/>
 <layers>
 <layer number="1" name="Top" color="4" fill="1" visible="no" active="no"/>
@@
 <part name="U1" library="HM-10_BLE" deviceset="HM-10" device=""/>
 <part name="U$1" library="SparkFun-RF" deviceset="XBEE-1" device="B1"/>
+<part name="RXD" library="SparkFun-LED" deviceset="LED-GREEN" device="0603" value="GREEN"/>
+<part name="TXD" library="SparkFun-LED" deviceset="LED-GREEN" device="0603" value="RED"/>
+<part name="R1" library="SparkFun-Resistors" deviceset="0.3OHM-1/8W-1%(0805)" device="" value="470R"/>
+<part name="R2" library="SparkFun-Resistors" deviceset="0.3OHM-1/8W-1%(0805)" device="" value="470R"/>
+<part name="GND1" library="SparkFun-Aesthetics" deviceset="GND" device=""/>
+<part name="GND2" library="SparkFun-Aesthetics" deviceset="GND" device=""/>
+<part name="R3" library="SparkFun-Resistors" deviceset="0.3OHM-1/8W-1%(0805)" device="" value="470R"/>
+<part name="R4" library="SparkFun-Resistors" deviceset="0.3OHM-1/8W-1%(0805)" device="" value="470R"/>
+<part name="D1" library="SparkFun-LED" deviceset="LED-BLUE" device="0603" value="BLUE"/>
+<part name="GND" library="SparkFun-Aesthetics" deviceset="GND" device=""/>
 </parts>
 <sheets>
 <sheet>
+<description>HM-10 XBee Breakout</description>
 <plain>
 </plain>
@@
 <instance part="U1" gate="G$1" x="181.61" y="138.43"/>
 <instance part="U$1" gate="G$1" x="116.84" y="143.51"/>
+<instance part="RXD" gate="G$1" x="107.95" y="175.26" rot="R90"/>
+<instance part="TXD" gate="G$1" x="107.95" y="165.1" rot="R90"/>
+<instance part="R1" gate="G$1" x="96.52" y="175.26"/>
+<instance part="R2" gate="G$1" x="96.52" y="165.1"/>
+<instance part="GND1" gate="1" x="118.11" y="162.56"/>
+<instance part="GND2" gate="1" x="118.11" y="172.72"/>
+<instance part="R3" gate="G$1" x="218.44" y="135.89"/>
+<instance part="R4" gate="G$1" x="218.44" y="120.65"/>
+<instance part="D1" gate="G$1" x="233.68" y="135.89" rot="R90"/>
+<instance part="GND" gate="1" x="246.38" y="133.35"/>
 </instances>
 <busses>
@@
 <label x="191.77" y="109.22" size="1.778" layer="95"/>
 </segment>
+<segment>
+<pinref part="TXD" gate="G$1" pin="C"/>
+<wire x1="113.03" y1="165.1" x2="118.11" y2="165.1" width="0.1524" layer="91"/>
+<pinref part="GND1" gate="1" pin="GND"/>
+</segment>
+<segment>
+<pinref part="RXD" gate="G$1" pin="C"/>
+<wire x1="113.03" y1="175.26" x2="118.11" y2="175.26" width="0.1524" layer="91"/>
+<pinref part="GND2" gate="1" pin="GND"/>
+</segment>
+<segment>
+<pinref part="D1" gate="G$1" pin="C"/>
+<pinref part="GND" gate="1" pin="GND"/>
+<wire x1="238.76" y1="135.89" x2="246.38" y2="135.89" width="0.1524" layer="91"/>
+</segment>
+<segment>
+<pinref part="U1" gate="G$1" pin="GND@4"/>
+<wire x1="201.93" y1="130.81" x2="205.74" y2="130.81" width="0.1524" layer="91"/>
+<label x="204.47" y="130.81" size="1.778" layer="95"/>
+</segment>
 </net>
 <net name="VDD" class="0">
@@
 <label x="156.21" y="133.35" size="1.778" layer="95"/>
 </segment>
-</net>
+<segment>
+<pinref part="R4" gate="G$1" pin="2"/>
+<wire x1="223.52" y1="120.65" x2="232.41" y2="120.65" width="0.1524" layer="91"/>
+<label x="228.6" y="120.65" size="1.778" layer="95"/>
+</segment>
+</net>
+<net name="TX" class="0">
+<segment>
+<pinref part="U1" gate="G$1" pin="P1_6"/>
+<wire x1="161.29" y1="161.29" x2="156.21" y2="161.29" width="0.1524" layer="91"/>
+<label x="156.21" y="161.29" size="1.778" layer="95"/>
+</segment>
+<segment>
+<pinref part="U$1" gate="G$1" pin="DIN"/>
+<wire x1="96.52" y1="148.59" x2="91.44" y2="148.59" width="0.1524" layer="91"/>
+<label x="91.44" y="148.59" size="1.778" layer="95"/>
+</segment>
+<segment>
+<pinref part="R2" gate="G$1" pin="1"/>
+<wire x1="91.44" y1="165.1" x2="86.36" y2="165.1" width="0.1524" layer="91"/>
+<label x="86.36" y="165.1" size="1.778" layer="95"/>
+</segment>
+</net>
+<net name="RX" class="0">
+<segment>
+<pinref part="U1" gate="G$1" pin="P1_7"/>
+<wire x1="161.29" y1="158.75" x2="156.21" y2="158.75" width="0.1524" layer="91"/>
+<label x="156.21" y="158.75" size="1.778" layer="95"/>
+</segment>
+<segment>
+<pinref part="U$1" gate="G$1" pin="DOUT"/>
+<wire x1="96.52" y1="151.13" x2="91.44" y2="151.13" width="0.1524" layer="91"/>
+<label x="91.44" y="151.13" size="1.778" layer="95"/>
+</segment>
+<segment>
+<pinref part="R1" gate="G$1" pin="1"/>
+<wire x1="91.44" y1="175.26" x2="86.36" y2="175.26" width="0.1524" layer="91"/>
+<label x="86.36" y="175.26" size="1.778" layer="95"/>
+</segment>
+</net>
+<net name="N$1" class="0">
+<segment>
+<pinref part="R2" gate="G$1" pin="2"/>
+<pinref part="TXD" gate="G$1" pin="A"/>
+<wire x1="101.6" y1="165.1" x2="105.41" y2="165.1" width="0.1524" layer="91"/>
+</segment>
+</net>
+<net name="N$2" class="0">
+<segment>
+<pinref part="R1" gate="G$1" pin="2"/>
+<pinref part="RXD" gate="G$1" pin="A"/>
+<wire x1="101.6" y1="175.26" x2="105.41" y2="175.26" width="0.1524" layer="91"/>
+</segment>
+</net>
+<net name="N$3" class="0">
+<segment>
+<pinref part="R3" gate="G$1" pin="2"/>
+<pinref part="D1" gate="G$1" pin="A"/>
+<wire x1="223.52" y1="135.89" x2="231.14" y2="135.89" width="0.1524" layer="91"/>
+</segment>
+</net>
+<net name="N$4" class="0">
+<segment>
+<pinref part="U1" gate="G$1" pin="P1_2"/>
+<pinref part="R3" gate="G$1" pin="1"/>
+<wire x1="201.93" y1="135.89" x2="213.36" y2="135.89" width="0.1524" layer="91"/>
+</segment>
+</net>
+<net name="N$5" class="0">
+<segment>
+<pinref part="U1" gate="G$1" pin="P1_3"/>
+<wire x1="201.93" y1="133.35" x2="213.36" y2="133.35" width="0.1524" layer="91"/>
+<pinref part="R4" gate="G$1" pin="1"/>
+<wire x1="213.36" y1="133.35" x2="213.36" y2="120.65" width="0.1524" layer="91"/>
+</segment>
+</net>

Commit message: first working routing
Parts:
- removed D1: BLUE, SparkFun-LED:LED-BLUE0603
- added PWR: BLU, adafruit:LEDCHIPLED_0805
- RXD: value GREEN -> GRN; device SparkFun-LED:LED-GREEN0603 -> adafruit:LEDCHIPLED_0805
- TXD: device SparkFun-LED:LED-GREEN0603 -> adafruit:LEDCHIPLED_0805
Connections:
- net GND: now also PWR.C; no longer D1.C
- net N$3: now also PWR.A; no longer D1.A

Commit message: added missing capacitor
Parts:
- added C1: 0.1uF, SparkFun-Capacitors:0.1UF-25V(+80/-20%)(0603)
Connections:
- net GND: now also C1.2
- net VDD: now also C1.1
Changed lines of the file:
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@@
 <grid distance="0.05" unitdist="inch" unit="inch" style="lines" multiple="1" display="no" altdistance="0.025" altunitdist="inch" altunit="inch"/>
 <layers>
-<layer number="1" name="Top" color="4" fill="1" visible="yes" active="no"/>
-<layer number="16" name="Bottom" color="1" fill="1" visible="yes" active="no"/>
-<layer number="17" name="Pads" color="2" fill="1" visible="yes" active="no"/>
-<layer number="18" name="Vias" color="2" fill="1" visible="yes" active="no"/>
-<layer number="19" name="Unrouted" color="6" fill="1" visible="yes" active="no"/>
-<layer number="20" name="Dimension" color="15" fill="1" visible="yes" active="no"/>
-<layer number="21" name="tPlace" color="7" fill="1" visible="yes" active="no"/>
-<layer number="22" name="bPlace" color="7" fill="1" visible="yes" active="no"/>
-<layer number="23" name="tOrigins" color="15" fill="1" visible="yes" active="no"/>
-<layer number="24" name="bOrigins" color="15" fill="1" visible="yes" active="no"/>
-<layer number="25" name="tNames" color="7" fill="1" visible="yes" active="no"/>
-<layer number="26" name="bNames" color="7" fill="1" visible="yes" active="no"/>
-<layer number="27" name="tValues" color="7" fill="1" visible="yes" active="no"/>
-<layer number="28" name="bValues" color="7" fill="1" visible="yes" active="no"/>
+<layer number="1" name="Top" color="4" fill="1" visible="no" active="no"/>
+<layer number="16" name="Bottom" color="1" fill="1" visible="no" active="no"/>
+<layer number="17" name="Pads" color="2" fill="1" visible="no" active="no"/>
+<layer number="18" name="Vias" color="2" fill="1" visible="no" active="no"/>
+<layer number="19" name="Unrouted" color="6" fill="1" visible="no" active="no"/>
+<layer number="20" name="Dimension" color="15" fill="1" visible="no" active="no"/>
+<layer number="21" name="tPlace" color="7" fill="1" visible="no" active="no"/>
+<layer number="22" name="bPlace" color="7" fill="1" visible="no" active="no"/>
+<layer number="23" name="tOrigins" color="15" fill="1" visible="no" active="no"/>
+<layer number="24" name="bOrigins" color="15" fill="1" visible="no" active="no"/>
+<layer number="25" name="tNames" color="7" fill="1" visible="no" active="no"/>
+<layer number="26" name="bNames" color="7" fill="1" visible="no" active="no"/>
+<layer number="27" name="tValues" color="7" fill="1" visible="no" active="no"/>
+<layer number="28" name="bValues" color="7" fill="1" visible="no" active="no"/>
 <layer number="29" name="tStop" color="7" fill="3" visible="no" active="no"/>
 <layer number="30" name="bStop" color="7" fill="6" visible="no" active="no"/>
@@
 <layer number="35" name="tGlue" color="7" fill="4" visible="no" active="no"/>
 <layer number="36" name="bGlue" color="7" fill="5" visible="no" active="no"/>
-<layer number="37" name="tTest" color="7" fill="1" visible="yes" active="no"/>
-<layer number="38" name="bTest" color="7" fill="1" visible="yes" active="no"/>
+<layer number="37" name="tTest" color="7" fill="1" visible="no" active="no"/>
+<layer number="38" name="bTest" color="7" fill="1" visible="no" active="no"/>
 <layer number="39" name="tKeepout" color="4" fill="11" visible="no" active="no"/>
 <layer number="40" name="bKeepout" color="1" fill="11" visible="no" active="no"/>
@@
 <layer number="44" name="Drills" color="7" fill="1" visible="no" active="no"/>
 <layer number="45" name="Holes" color="7" fill="1" visible="no" active="no"/>
-<layer number="46" name="Milling" color="3" fill="1" visible="yes" active="no"/>
-<layer number="47" name="Measures" color="7" fill="1" visible="yes" active="no"/>
-<layer number="48" name="Document" color="7" fill="1" visible="yes" active="no"/>
-<layer number="49" name="Reference" color="7" fill="1" visible="yes" active="no"/>
-<layer number="50" name="dxf" color="7" fill="1" visible="yes" active="no"/>
-<layer number="51" name="tDocu" color="7" fill="1" visible="yes" active="no"/>
-<layer number="52" name="bDocu" color="7" fill="1" visible="yes" active="no"/>
-<layer number="53" name="tGND_GNDA" color="7" fill="9" visible="yes" active="no"/>
-<layer number="54" name="bGND_GNDA" color="1" fill="9" visible="yes" active="no"/>
-<layer number="56" name="wert" color="7" fill="1" visible="yes" active="no"/>
+<layer number="46" name="Milling" color="3" fill="1" visible="no" active="no"/>
+<layer number="47" name="Measures" color="7" fill="1" visible="no" active="no"/>
+<layer number="48" name="Document" color="7" fill="1" visible="no" active="no"/>
+<layer number="49" name="Reference" color="7" fill="1" visible="no" active="no"/>
+<layer number="50" name="dxf" color="7" fill="1" visible="no" active="no"/>
+<layer number="51" name="tDocu" color="7" fill="1" visible="no" active="no"/>
+<layer number="52" name="bDocu" color="7" fill="1" visible="no" active="no"/>
+<layer number="53" name="tGND_GNDA" color="7" fill="9" visible="no" active="no"/>
+<layer number="54" name="bGND_GNDA" color="1" fill="9" visible="no" active="no"/>
+<layer number="56" name="wert" color="7" fill="1" visible="no" active="no"/>
 <layer number="57" name="tCAD" color="7" fill="1" visible="no" active="no"/>
 <layer number="91" name="Nets" color="2" fill="1" visible="yes" active="yes"/>
@@
 <part name="PWR" library="adafruit" deviceset="LED" device="CHIPLED_0805" value="BLU"/>
 <part name="GND3" library="SparkFun-Aesthetics" deviceset="GND" device=""/>
+<part name="C1" library="SparkFun-Capacitors" deviceset="0.1UF-25V(+80/-20%)(0603)" device="" value="0.1uF"/>
+<part name="GND4" library="SparkFun-Aesthetics" deviceset="GND" device=""/>
 </parts>
 <sheets>
@@
 <instance part="PWR" gate="G$1" x="233.68" y="135.89" rot="R90"/>
 <instance part="GND3" gate="1" x="247.65" y="133.35"/>
+<instance part="C1" gate="G$1" x="147.32" y="113.03"/>
+<instance part="GND4" gate="1" x="147.32" y="100.33"/>
 </instances>
 <busses>
@@
 <junction x="247.65" y="135.89"/>
 </segment>
+<segment>
+<pinref part="C1" gate="G$1" pin="2"/>
+<wire x1="147.32" y1="110.49" x2="147.32" y2="102.87" width="0.1524" layer="91"/>
+<pinref part="GND4" gate="1" pin="GND"/>
+<wire x1="147.32" y1="102.87" x2="147.32" y2="101.6" width="0.1524" layer="91"/>
+<junction x="147.32" y="102.87"/>
+</segment>
 </net>
 <net name="VDD" class="0">
@@
 <wire x1="162.56" y1="133.35" x2="161.29" y2="133.35" width="0.1524" layer="91"/>
 <pinref part="U1" gate="G$1" pin="3.3V"/>
-<wire x1="161.29" y1="133.35" x2="156.21" y2="133.35" width="0.1524" layer="91"/>
-<junction x="161.29" y="133.35"/>
-<label x="156.21" y="133.35" size="1.778" layer="95"/>
-</segment>
-<segment>
+<pinref part="C1" gate="G$1" pin="1"/>
+<wire x1="147.32" y1="118.11" x2="147.32" y2="133.35" width="0.1524" layer="91"/>
+<wire x1="147.32" y1="133.35" x2="147.32" y2="144.78" width="0.1524" layer="91"/>
+<wire x1="161.29" y1="133.35" x2="147.32" y2="133.35" width="0.1524" layer="91"/>
+<junction x="147.32" y="133.35"/>
+<label x="152.4" y="133.35" size="1.778" layer="95"/>
+<label x="147.32" y="142.24" size="1.778" layer="95"/>
+</segment>
+<segment>

Commit message: Fixed RX/TX being backwards and removed the RX/TX LEDs
Parts:
- removed R1, R2: 470R, SparkFun-Resistors:0.3OHM-1/8W-1%(0805)
- removed RXD: GRN, adafruit:LEDCHIPLED_0805
- removed TXD: RED, adafruit:LEDCHIPLED_0805
Connections:
- removed net N$1: R2.2, TXD.A
- removed net N$2: R1.2, RXD.A
- net GND: no longer RXD.C, TXD.C
- net RX: now also U1.P1_6; no longer R1.1, U1.P1_7
- net TX: now also U1.P1_7; no longer R2.1, U1.P1_6
Changed lines of the file:
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@@
 <setting verticaltext="up"/>
 </settings>
-<grid distance="0.05" unitdist="inch" unit="inch" style="lines" multiple="1" display="no" altdistance="0.025" altunitdist="inch" altunit="inch"/>
+<grid distance="0.1" unitdist="inch" unit="inch" style="lines" multiple="1" display="no" altdistance="0.01" altunitdist="inch" altunit="inch"/>
 <layers>
 <layer number="1" name="Top" color="4" fill="1" visible="no" active="no"/>
@@
 <part name="U1" library="HM-10_BLE" deviceset="HM-10" device=""/>
 <part name="U$1" library="SparkFun-RF" deviceset="XBEE-1" device="B1"/>
-<part name="R1" library="SparkFun-Resistors" deviceset="0.3OHM-1/8W-1%(0805)" device="" value="470R"/>
-<part name="R2" library="SparkFun-Resistors" deviceset="0.3OHM-1/8W-1%(0805)" device="" value="470R"/>
-<part name="GND1" library="SparkFun-Aesthetics" deviceset="GND" device=""/>
-<part name="GND2" library="SparkFun-Aesthetics" deviceset="GND" device=""/>
 <part name="R3" library="SparkFun-Resistors" deviceset="0.3OHM-1/8W-1%(0805)" device="" value="470R"/>
 <part name="R4" library="SparkFun-Resistors" deviceset="0.3OHM-1/8W-1%(0805)" device="" value="470R"/>
-<part name="RXD" library="adafruit" deviceset="LED" device="CHIPLED_0805" value="GRN"/>
-<part name="TXD" library="adafruit" deviceset="LED" device="CHIPLED_0805" value="RED"/>
 <part name="PWR" library="adafruit" deviceset="LED" device="CHIPLED_0805" value="BLU"/>
 <part name="GND3" library="SparkFun-Aesthetics" deviceset="GND" device=""/>
@@
 <instance part="U1" gate="G$1" x="181.61" y="138.43"/>
 <instance part="U$1" gate="G$1" x="116.84" y="143.51"/>
-<instance part="R1" gate="G$1" x="96.52" y="175.26"/>
-<instance part="R2" gate="G$1" x="96.52" y="165.1"/>
-<instance part="GND1" gate="1" x="118.11" y="162.56"/>
-<instance part="GND2" gate="1" x="118.11" y="172.72"/>
 <instance part="R3" gate="G$1" x="218.44" y="135.89"/>
 <instance part="R4" gate="G$1" x="218.44" y="120.65"/>
-<instance part="RXD" gate="G$1" x="107.95" y="175.26" rot="R90"/>
-<instance part="TXD" gate="G$1" x="107.95" y="165.1" rot="R90"/>
 <instance part="PWR" gate="G$1" x="233.68" y="135.89" rot="R90"/>
 <instance part="GND3" gate="1" x="247.65" y="133.35"/>
@@
 </segment>
 <segment>
-<wire x1="113.03" y1="165.1" x2="118.11" y2="165.1" width="0.1524" layer="91"/>
-<pinref part="GND1" gate="1" pin="GND"/>
-<pinref part="TXD" gate="G$1" pin="C"/>
-<junction x="118.11" y="165.1"/>
-</segment>
-<segment>
-<wire x1="113.03" y1="175.26" x2="118.11" y2="175.26" width="0.1524" layer="91"/>
-<pinref part="GND2" gate="1" pin="GND"/>
-<pinref part="RXD" gate="G$1" pin="C"/>
-<junction x="118.11" y="175.26"/>
-</segment>
-<segment>
 <pinref part="U1" gate="G$1" pin="GND@4"/>
 <wire x1="201.93" y1="130.81" x2="205.74" y2="130.81" width="0.1524" layer="91"/>
@@
 <net name="TX" class="0">
 <segment>
+<pinref part="U$1" gate="G$1" pin="DIN"/>
+<wire x1="96.52" y1="148.59" x2="91.44" y2="148.59" width="0.1524" layer="91"/>
+<label x="91.44" y="148.59" size="1.778" layer="95"/>
+</segment>
+<segment>
+<pinref part="U1" gate="G$1" pin="P1_7"/>
+<wire x1="161.29" y1="158.75" x2="156.21" y2="158.75" width="0.1524" layer="91"/>
+<label x="156.21" y="158.75" size="1.778" layer="95"/>
+</segment>
+</net>
+<net name="RX" class="0">
+<segment>
+<pinref part="U$1" gate="G$1" pin="DOUT"/>
+<wire x1="96.52" y1="151.13" x2="91.44" y2="151.13" width="0.1524" layer="91"/>
+<label x="91.44" y="151.13" size="1.778" layer="95"/>
+</segment>
+<segment>
 <pinref part="U1" gate="G$1" pin="P1_6"/>
 <wire x1="161.29" y1="161.29" x2="156.21" y2="161.29" width="0.1524" layer="91"/>
 <label x="156.21" y="161.29" size="1.778" layer="95"/>
 </segment>
-<segment>
-<pinref part="U$1" gate="G$1" pin="DIN"/>
-<wire x1="96.52" y1="148.59" x2="91.44" y2="148.59" width="0.1524" layer="91"/>
-<label x="91.44" y="148.59" size="1.778" layer="95"/>
-</segment>
-<segment>
-<pinref part="R2" gate="G$1" pin="1"/>
-<wire x1="91.44" y1="165.1" x2="86.36" y2="165.1" width="0.1524" layer="91"/>
-<label x="86.36" y="165.1" size="1.778" layer="95"/>
-</segment>
-</net>
-<net name="RX" class="0">
-<segment>
-<pinref part="U1" gate="G$1" pin="P1_7"/>
-<wire x1="161.29" y1="158.75" x2="156.21" y2="158.75" width="0.1524" layer="91"/>
-<label x="156.21" y="158.75" size="1.778" layer="95"/>
-</segment>
-<segment>
-<pinref part="U$1" gate="G$1" pin="DOUT"/>
-<wire x1="96.52" y1="151.13" x2="91.44" y2="151.13" width="0.1524" layer="91"/>
-<label x="91.44" y="151.13" size="1.778" layer="95"/>
-</segment>
-<segment>
-<pinref part="R1" gate="G$1" pin="1"/>
-<wire x1="91.44" y1="175.26" x2="86.36" y2="175.26" width="0.1524" layer="91"/>
-<label x="86.36" y="175.26" size="1.778" layer="95"/>
-</segment>
-</net>
-<net name="N$1" class="0">
-<segment>
-<pinref part="R2" gate="G$1" pin="2"/>
-<wire x1="101.6" y1="165.1" x2="105.41" y2="165.1" width="0.1524" layer="91"/>
-<pinref part="TXD" gate="G$1" pin="A"/>
-</segment>
-</net>
-<net name="N$2" class="0">
-<segment>
-<pinref part="R1" gate="G$1" pin="2"/>
-<wire x1="101.6" y1="175.26" x2="105.41" y2="175.26" width="0.1524" layer="91"/>
-<pinref part="RXD" gate="G$1" pin="A"/>
-</segment>
-</net>
+</net>
